File: Main Processing Board V2/Main Processing Board V2.kicad_pcb (KiCad board)
At the start: 2 copper layers, 37.3 x 37.8 mm, 22 parts, among them J1 Conn_01x10_MountingPin, J4 Conn_01x06_MountingPin, U2 LSM6DSOXTR, U3 Seeed Studio RA4M1, U4 MS5611-01BA03, U5 MMC5603NJ

Commit message: added BOM work
Parts:
- added G***: LOGO, project-library:silkLogo, B.Cu at (159.5, 96.1)
Connections:
- U2 pad 2: unconnected-(U2-SDX-Pad2) -> GND
- U2 pad 3: unconnected-(U2-SCX-Pad3) -> GND
Routing:
- net GND: track 25.3 -> 23.0 mm
Other:
- board text added: "BYU POCKETQUBE 2026 MAIN BOARD REV: X1"
- board text added: "If Found Please Contact spacecraftclub@byu.edu"
