File: Main Processing Board V2/Main Processing Board V2.kicad_sch (KiCad schematic)
At the start: 21 parts, among them J1 Conn_01x10_MountingPin, J4 Conn_01x06_MountingPin, U2 LSM6DSOXTR, U3 Seeed Studio RA4M1, U4 MS5611-01BA03, U5 MMC5603NJ

Commit message: added BOM work
Connections:
- net GND: now also U2.2 (SDX), U2.3 (SCX)
- no-connect marks 29 -> 27
Changed lines of the file:
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@@
+	)
+	(junction
+		(at 266.7 34.29)
+		(diameter 0)
+		(color 0 0 0 0)
 	)
 	(junction
@@
 	)
 	(junction
+		(at 266.7 36.83)
+		(diameter 0)
+		(color 0 0 0 0)
+	)
+	(junction
 		(at 265.43 26.67)
 		(diameter 0)
@@
 	)
 	(no_connect
-		(at 262.89 39.37)
-	)
-	(no_connect
 		(at 97.79 58.42)
 	)
@@
 	)
 	(no_connect
-		(at 262.89 36.83)
-	)
-	(no_connect
 		(at 69.85 72.39)
 	)
@@
 	(wire
 		(pts
+			(xy 266.7 34.29) (xy 270.51 34.29)
+		)
+		(stroke
+			(width 0)
+			(type default)
+		)
+	)
+	(wire
+		(pts
 			(xy 85.09 134.62) (xy 69.85 134.62)
 		)
@@
 	(wire
 		(pts
+			(xy 266.7 39.37) (xy 262.89 39.37)
+		)
+		(stroke
+			(width 0)
+			(type default)
+		)
+	)
+	(wire
+		(pts
 			(xy 262.89 54.61) (xy 270.51 54.61)
 		)
@@
 	(wire
 		(pts
+			(xy 266.7 36.83) (xy 266.7 39.37)
+		)
+		(stroke
+			(width 0)
+			(type default)
+		)
+	)
+	(wire
+		(pts
 			(xy 270.51 54.61) (xy 270.51 55.88)
 		)
@@
 	(wire
 		(pts
-			(xy 262.89 34.29) (xy 270.51 34.29)
+			(xy 262.89 34.29) (xy 266.7 34.29)
 		)
 		(stroke
@@
 	(wire
 		(pts
+			(xy 262.89 36.83) (xy 266.7 36.83)
+		)
+		(stroke
+			(width 0)
+			(type default)
+		)
+	)
+	(wire
+		(pts
 			(xy 273.05 27.94) (xy 273.05 25.4)
 		)
@@
 		)
 		(stroke
+			(width 0)
+			(type default)
+		)
+	)
+	(wire
+		(pts
+			(xy 266.7 34.29) (xy 266.7 36.83)
+		)
+		(stroke
